Commit message: feat: Add sensor fusion

File: tr_description/urdf/amr.urdf (robot description, URDF)
Before this commit: robot amr, 4 links, 3 joints
Links:
- added link imu_link
Joints:
- removed joint scan1
- removed joint scan2
- added joint imu_joint: type fixed, parent base_link, child imu_link, origin xyz=0.189 -0.041 0.094 rpy=0 0 0
- added joint scan1_joint: type fixed, parent base_link, child scan1, origin xyz=0.350 0.225 0.0505 rpy=0.0 0.0 0.785398
- added joint scan2_joint: type fixed, parent base_link, child scan2, origin xyz=-0.350 -0.225 0.0505 rpy=0.0 0.0 3.92699
