Commit message: Fix sim parameters

File: tr_description/urdf/amr_body.urdf.xacro (robot description, xacro)
@@ -184,14 +184,4 @@
         <axis xyz="0.0 0.0 -1.0" />
     </joint>
-    <transmission name="wheel_left_joint_transmission">
-        <type>transmission_interface/SimpleTransmission</type>
-        <joint name="wheel_left_joint">
-            <hardwareInterface>VelocityJointInterface</hardwareInterface>
-        </joint>
-        <actuator name="wheel_left_joint_motor">
-            <hardwareInterface>VelocityJointInterface</hardwareInterface>
-            <mechanicalReduction>1</mechanicalReduction>
-        </actuator>
-    </transmission>
     <link name="wheel_right">
         <inertial>
@@ -220,14 +210,4 @@
         <axis xyz="0.0 0.0 1.0" />
     </joint>
-    <transmission name="wheel_right_joint_transmission">
-        <type>transmission_interface/SimpleTransmission</type>
-        <joint name="wheel_right_joint">
-            <hardwareInterface>VelocityJointInterface</hardwareInterface>
-        </joint>
-        <actuator name="wheel_right_joint_motor">
-            <hardwareInterface>VelocityJointInterface</hardwareInterface>
-            <mechanicalReduction>1</mechanicalReduction>
-        </actuator>
-    </transmission>
     <link name="caster_fork_front_left">
         <inertial>

Commit message: Add OpenArm description

File: tr_description/urdf/amr_body.urdf.xacro (robot description, xacro)
@@ -1,4 +1,5 @@
 <?xml version='1.0' encoding='utf-8'?>
-<robot name="amr">
+<robot name="amr" xmlns:xacro="http://www.ros.org/wiki/xacro">
+    <xacro:arg name="use_arm" default="false"/>
     <link name="base_footprint"/>
     <link name="base_link">
@@ -22,5 +23,5 @@
     </link>
     <joint name="base_link_joint" type="fixed">
-        <origin xyz="0 0 0" rpy="0 0 0"/>
+        <origin xyz="0 0 3" rpy="0 0 0"/>
         <parent link="base_footprint"/>
         <child  link="base_link"/>
@@ -418,3 +419,7 @@
         <axis xyz="0.0 0.0 1.0" />
     </joint>
+    <xacro:include filename="openarm_bimanual_sim.urdf.xacro" />
+    <xacro:if value="$(arg use_arm)">
+        <xacro:amr_dual_arm />
+    </xacro:if>
 </robot>

File: tr_description/urdf/amr_gazebo.urdf.xacro (robot description, xacro)
@@ -36,19 +36,4 @@
         visualize="false"
     />
-    <ros2_control name="GazeboSystem" type="system">
-        <hardware>
-            <plugin>gazebo_ros2_control/GazeboSystem</plugin>
-        </hardware>
-        <joint name="wheel_left_joint">
-            <command_interface name="velocity"/>
-            <state_interface name="position"/>
-            <state_interface name="velocity"/>
-        </joint>
-        <joint name="wheel_right_joint">
-            <command_interface name="velocity"/>
-            <state_interface name="position"/>
-            <state_interface name="velocity"/>
-        </joint>
-    </ros2_control>
     <gazebo>
         <plugin filename="libgazebo_ros2_control.so" name="gazebo_ros2_control">

File: tr_description/urdf/amr_sim.urdf.xacro (robot description, xacro)
@@ -4,4 +4,6 @@
     <!--set use_gazebo = false for implementation on real robot-->
     <xacro:arg name="use_gazebo" default="true"/>
+    <xacro:arg name="use_arm" default="false"/>
+    <xacro:include filename="$(find tr_description)/urdf/openarm.ros2_control.xacro" />
     <!-- import main body description -->
     <xacro:include filename="amr_body.urdf.xacro"/>
@@ -9,4 +11,28 @@
     <xacro:if value="$(arg use_gazebo)">
         <xacro:include filename="amr_gazebo.urdf.xacro"/>
+        <ros2_control name="GazeboSystem" type="system">
+            <hardware>
+                <plugin>gazebo_ros2_control/GazeboSystem</plugin>
+            </hardware>
+            <joint name="wheel_left_joint">
+                <command_interface name="velocity"/>
+                <state_interface name="position"/>
+                <state_interface name="velocity"/>
+            </joint>
+            <joint name="wheel_right_joint">
+                <command_interface name="velocity"/>
+                <state_interface name="position"/>
+                <state_interface name="velocity"/>
+            </joint>
+            <joint name="wheel_right_joint">
+                <command_interface name="velocity"/>
+                <state_interface name="position"/>
+                <state_interface name="velocity"/>
+            </joint>
+            <xacro:if value="$(arg use_arm)">
+                <xacro:single_arm_control prefix="openarm_left" />
+                <xacro:single_arm_control prefix="openarm_right" />
+            </xacro:if>
+        </ros2_control>
     </xacro:if>
 </robot>
